File: hardware/v2/SHS-Z2M-Presence-v2.kicad_pcb (KiCad board)
At the start: 4 copper layers, 39 x 49 mm, 28 parts, among them J1 USB_C_Receptacle, SW1 RESET, SW2 BOOT, U1 ESP32-C6-WROOM-1-N8, U2 LD2410C, U3 LD2450, U4 AP2112K-3.3, U5 USBLC6-2SC6

Commit message: Fix schematic wire gaps and restore PCB zone nets
Schematic fixes:
- Fix SW1/SW2 wire endpoints (0.032mm gap: 98.952→98.92, etc.)
  Both switches now correctly connect to ESP_EN/BOOT and GND
- Replace SW1-to-ESP_EN wire through C8 GND area with direct
  ESP_EN label (avoids T-junction short with GND)
- Add direct +5V label on U4.EN wire (avoids T-junction
  dependency through IN pin at same x-coordinate)

PCB fixes:
- Restore zone net assignments stripped during net cleanup:
  F.Cu=GND, B.Cu=GND, In1.Cu=GND, In2.Cu=+3V3

Co-Authored-By: Claude Opus 4.6 <noreply@anthropic.com>
Routing:
- added copper zone on In2.Cu, net +3V3
- added copper zone on B.Cu, net GND
- added copper zone on F.Cu, net GND
- added copper zone on In1.Cu, net GND
- removed copper zone on B.Cu, net (none)
- removed copper zone on F.Cu, net (none)
- removed copper zone on In1.Cu, net (none)
- removed copper zone on In2.Cu, net (none)
Changed lines of the file:
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@@
 	)
 	(zone
+		(net "GND")
 		(layer "F.Cu")
 		(hatch edge 0.508)
@@
 	)
 	(zone
+		(net "GND")
 		(layer "B.Cu")
 		(hatch edge 0.508)
@@
 	)
 	(zone
+		(net "GND")
 		(layer "In1.Cu")
 		(uuid "a1b2c3d4-in1g-4lay-gnd0-000000000001")
@@
 	)
 	(zone
+		(net "+3V3")
 		(layer "In2.Cu")
 		(uuid "a1b2c3d4-in2p-4lay-pwr0-000000000001")
